File: modules/button_module/button_module.sch (KiCad schematic (older format))
At the start: 8 parts, among them J1 Conn_02x03_Counter_Clockwise, U1 ATtiny85-20PU

Commit message: Changes
Parts:
- removed D1, D2, D3: LED, LED_THT:LED_D3.0mm, symbol Device:LED
- removed R2, R3: 220, Resistor_SMD:R_0805_2012Metric_Pad1.20x1.40mm_HandSolder, symbol Device:R
- added SW1: SW_SPST, Button_Switch_THT:SW_PUSH_6mm, symbol Switch:SW_SPST
- R1: value 220 -> 100k
Connections:
- net LED1 is gone; now on net Intr: U1.6 (PB1)
- net LED2 is gone; now on an unnamed net: U1.2 (XTAL1/PB3)
- net +3V3: now also R1.1
- net GND: now also SW1.2 (B); no longer R1.1
- net Intr: now reaches J1.3 (Pin_3)
- net at R1.2: now also SW1.1 (A)
- net LED3: no longer names the net of U1.3 (XTAL2/PB4)
Other:
- note removed: "Intr pin, not used with LEDS"
- note removed: "Leds"
Changed lines of the file:
@@
 $EndComp
-Wire Wire Line
-	4450 2450 4600 2450
 Wire Wire Line
 	4450 2350 4600 2350
@@
 Text Label 1150 2000 2    50   ~ 0
 SDA
-NoConn ~ 1400 2100
-Text Notes 650  2250 0    50   ~ 0
-Intr pin, not used with LEDS
 Text Label 4600 2150 0    50   ~ 0
 SDA
@@
 SCL
 Text Label 4600 2250 0    50   ~ 0
-LED1
-Text Label 4600 2450 0    50   ~ 0
-LED2
+Intr
+$Comp
+L Switch:SW_SPST SW1
+U 1 1 60BE0F93
+P 5200 2450
+F 0 "SW1" H 5200 2685 50  0000 C CNN
+F 1 "SW_SPST" H 5200 2594 50  0000 C CNN
+F 2 "Button_Switch_THT:SW_PUSH_6mm" H 5200 2450 50  0001 C CNN
+F 3 "~" H 5200 2450 50  0001 C CNN
+	1    5200 2450
+	1    0    0    -1
+$EndComp
+Text Label 1150 2100 2    50   ~ 0
+Intr
+Wire Wire Line
+	1400 2100 1150 2100
+Wire Wire Line
+	5400 2450 5550 2450
+Wire Wire Line
+	5550 2450 5550 2500
+$Comp
+L power:GND #PWR?
+U 1 1 60BE55BC
+P 5550 2500
+F 0 "#PWR?" H 5550 2250 50  0001 C CNN
+F 1 "GND" H 5555 2327 50  0000 C CNN
+F 2 "" H 5550 2500 50  0001 C CNN
+F 3 "" H 5550 2500 50  0001 C CNN
+	1    5550 2500
+	1    0    0    -1
+$EndComp
+NoConn ~ 4600 2550
 Wire Wire Line
 	4450 2550 4600 2550
-Text Label 4600 2550 0    50   ~ 0
-LED3
 Wire Wire Line
-	5850 2200 6050 2200
+	4900 2450 5000 2450
+Wire Wire Line
+	4450 2450 4900 2450
+Connection ~ 4900 2450
+Wire Wire Line
+	4900 2450 4900 2300
 $Comp
-L Device:LED D1
-U 1 1 60BEFDCF
-P 6200 2200
-F 0 "D1" H 6193 1945 50  0000 C CNN
-F 1 "LED" H 6193 2036 50  0000 C CNN
-F 2 "LED_THT:LED_D3.0mm" H 6200 2200 50  0001 C CNN
-F 3 "~" H 6200 2200 50  0001 C CNN
-	1    6200 2200
-	-1   0    0    1
+L Device:R R1
+U 1 1 60BE5CA7
+P 4900 2150
+F 0 "R1" H 4970 2196 50  0000 L CNN
+F 1 "100k" H 4970 2105 50  0000 L CNN
+F 2 "Resistor_SMD:R_0805_2012Metric_Pad1.20x1.40mm_HandSolder" V 4830 2150 50  0001 C CNN
+F 3 "~" H 4900 2150 50  0001 C CNN
+	1    4900 2150
+	1    0    0    -1
 $EndComp
 Wire Wire Line
-	6350 2200 6550 2200
+	4900 2000 4900 1900
 $Comp
-L Device:R R1
-U 1 1 60BF0F2F
-P 6700 2200
-F 0 "R1" V 6493 2200 50  0000 C CNN
-F 1 "220" V 6584 2200 50  0000 C CNN
-F 2 "Resistor_SMD:R_0805_2012Metric_Pad1.20x1.40mm_HandSolder" V 6630 2200 50  0001 C CNN
-F 3 "~" H 6700 2200 50  0001 C CNN
-	1    6700 2200
-	0    1    1    0
+L power:+3V3 #PWR?
+U 1 1 60BE65AA
+P 4900 1900
+F 0 "#PWR?" H 4900 1750 50  0001 C CNN
+F 1 "+3V3" H 4915 2073 50  0000 C CNN
+F 2 "" H 4900 1900 50  0001 C CNN
+F 3 "" H 4900 1900 50  0001 C CNN
+	1    4900 1900
+	1    0    0    -1
 $EndComp
-Wire Wire Line
-	6850 2200 6950 2200
-$Comp
-L power:GND #PWR?
-U 1 1 60BF17AA
-P 6950 2200
-F 0 "#PWR?" H 6950 1950 50  0001 C CNN
-F 1 "GND" V 6955 2072 50  0000 R CNN
-F 2 "" H 6950 2200 50  0001 C CNN
-F 3 "" H 6950 2200 50  0001 C CNN
-	1    6950 2200
-	0    -1   -1   0
-$EndComp
-Text Label 5850 2200 0    50   ~ 0
-LED1
-Wire Wire Line
-	5850 2600 6050 2600
-$Comp
-L Device:LED D2
-U 1 1 60BF2701
-P 6200 2600
-F 0 "D2" H 6193 2345 50  0000 C CNN
-F 1 "LED" H 6193 2436 50  0000 C CNN
-F 2 "LED_THT:LED_D3.0mm" H 6200 2600 50  0001 C CNN
-F 3 "~" H 6200 2600 50  0001 C CNN
-	1    6200 2600
-	-1   0    0    1
-$EndComp
-Wire Wire Line
-	6350 2600 6550 2600
-$Comp
-L Device:R R2
-U 1 1 60BF2708
-P 6700 2600
-F 0 "R2" V 6493 2600 50  0000 C CNN
-F 1 "220" V 6584 2600 50  0000 C CNN
-F 2 "Resistor_SMD:R_0805_2012Metric_Pad1.20x1.40mm_HandSolder" V 6630 2600 50  0001 C CNN
-F 3 "~" H 6700 2600 50  0001 C CNN
-	1    6700 2600
-	0    1    1    0
-$EndComp
-Wire Wire Line
-	6850 2600 6950 2600
-$Comp
-L power:GND #PWR?
-U 1 1 60BF270F
-P 6950 2600
-F 0 "#PWR?" H 6950 2350 50  0001 C CNN
-F 1 "GND" V 6955 2472 50  0000 R CNN
-F 2 "" H 6950 2600 50  0001 C CNN
-F 3 "" H 6950 2600 50  0001 C CNN
-	1    6950 2600
-	0    -1   -1   0
-$EndComp
-Text Label 5850 2600 0    50   ~ 0
-LED2
-Wire Wire Line
-	5850 3000 6050 3000
-$Comp
-L Device:LED D3
-U 1 1 60BF2FBF
-P 6200 3000
-F 0 "D3" H 6193 2745 50  0000 C CNN
-F 1 "LED" H 6193 2836 50  0000 C CNN
-F 2 "LED_THT:LED_D3.0mm" H 6200 3000 50  0001 C CNN
-F 3 "~" H 6200 3000 50  0001 C CNN
-	1    6200 3000
-	-1   0    0    1
-$EndComp
-Wire Wire Line
-	6350 3000 6550 3000
-$Comp
-L Device:R R3
-U 1 1 60BF2FC6
-P 6700 3000
-F 0 "R3" V 6493 3000 50  0000 C CNN
-F 1 "220" V 6584 3000 50  0000 C CNN
-F 2 "Resistor_SMD:R_0805_2012Metric_Pad1.20x1.40mm_HandSolder" V 6630 3000 50  0001 C CNN
-F 3 "~" H 6700 3000 50  0001 C CNN
-	1    6700 3000
-	0    1    1    0
-$EndComp
-Wire Wire Line
-	6850 3000 6950 3000
-$Comp
-L power:GND #PWR?
-U 1 1 60BF2FCD
-P 6950 3000
-F 0 "#PWR?" H 6950 2750 50  0001 C CNN
-F 1 "GND" V 6955 2872 50  0000 R CNN
-F 2 "" H 6950 3000 50  0001 C CNN
-F 3 "" H 6950 3000 50  0001 C CNN
-	1    6950 3000
-	0    -1   -1   0
-$EndComp
-Text Label 5850 3000 0    50   ~ 0
-LED3
-Wire Notes Line
-	5800 1850 5800 3200
-Wire Notes Line
-	5800 3200 7350 3200
-Wire Notes Line
-	7350 3200 7350 1850
-Wire Notes Line
-	7350 1850 5800 1850
-Text Notes 5800 1800 0    50   ~ 0
-Leds
 $EndSCHEMATC
